Commit message: fix: Added RGBD camera

File: Project 4/my_robot/urdf/my_robot.xacro (robot description, xacro)
@@ -181,4 +181,6 @@
     <axis xyz="0 1 0" rpy="0 0 0"/>
   </joint>
+  <link name="camera_link_optical">
+  </link>
   <joint name="camera_optical_joint" type="fixed">
     <origin xyz="0 0 0" rpy="-1.5707 0 -1.5707"/>
@@ -186,6 +188,4 @@
     <child link="camera_link_optical"/>
   </joint>
-  <link name="camera_link_optical">
-  </link>
 <gazebo reference="left_wheel">
     <material>Gazebo/Purple</material>

Commit message: fix: Added camera_link_optical

File: Project 4/my_robot/urdf/my_robot.xacro (robot description, xacro)
@@ -182,9 +182,33 @@
   </joint>
   <link name="camera_link_optical">
+    <pose>0 0 0 0 0 0</pose>
+    <inertial>
+      <mass value="0.1"/>
+      <origin xyz="0.0 0 0" rpy=" 0 0 0"/>
+      <box_inertia m="0.1" x="0.05" y="0.05" z="0.05"/>
+      <inertia
+          ixx="1e-6" ixy="0" ixz="0"
+          iyy="1e-6" iyz="0"
+          izz="1e-6"
+      />
+    </inertial>
+    <collision name='collision'>
+      <origin xyz="0 0 0" rpy=" 0 0 0"/>
+      <geometry>
+        <box size=".05 .05 .05"/>
+      </geometry>
+    </collision>
+    <visual name='camera_optical_visual'>
+      <origin xyz="0 0 0" rpy=" 0 0 0"/>
+      <geometry>
+        <box size=".05 .05 .05"/>
+      </geometry>
+    </visual>
   </link>
   <joint name="camera_optical_joint" type="fixed">
-    <origin xyz="0 0 0" rpy="-1.5707 0 -1.5707"/>
-    <parent link="camera"/>
+    <origin xyz="0.2 0 0" rpy="-1.5707 0 -1.5707"/>
+    <parent link="chassis"/>
     <child link="camera_link_optical"/>
+    <axis xyz="0.0 1.0 0.0"/>
   </joint>
 <gazebo reference="left_wheel">
@@ -200,3 +224,6 @@
     <material>Gazebo/Blue</material>
 </gazebo>
+<gazebo reference="camera_link_optical">
+    <material>Gazebo/Yellow</material>
+</gazebo>
 </robot>

Commit message: fix: Small changes to urdf

File: Project 4/my_robot/urdf/my_robot.xacro (robot description, xacro)
@@ -181,35 +181,11 @@
     <axis xyz="0 1 0" rpy="0 0 0"/>
   </joint>
+  <joint name="camera_optical_joint" type="fixed">
+    <origin xyz="0 0 0" rpy="-1.5707 0 -1.5707"/>
+    <parent link="camera"/>
+    <child link="camera_link_optical"/>
+  </joint>
   <link name="camera_link_optical">
-    <pose>0 0 0 0 0 0</pose>
-    <inertial>
-      <mass value="0.1"/>
-      <origin xyz="0.0 0 0" rpy=" 0 0 0"/>
-      <box_inertia m="0.1" x="0.05" y="0.05" z="0.05"/>
-      <inertia
-          ixx="1e-6" ixy="0" ixz="0"
-          iyy="1e-6" iyz="0"
-          izz="1e-6"
-      />
-    </inertial>
-    <collision name='collision'>
-      <origin xyz="0 0 0" rpy=" 0 0 0"/>
-      <geometry>
-        <box size=".05 .05 .05"/>
-      </geometry>
-    </collision>
-    <visual name='camera_optical_visual'>
-      <origin xyz="0 0 0" rpy=" 0 0 0"/>
-      <geometry>
-        <box size=".05 .05 .05"/>
-      </geometry>
-    </visual>
-  </link>
-  <joint name="camera_optical_joint" type="fixed">
-    <origin xyz="0.2 0 0" rpy="-1.5707 0 -1.5707"/>
-    <parent link="chassis"/>
-    <child link="camera_link_optical"/>
-    <axis xyz="0.0 1.0 0.0"/>
-  </joint>
+  </link>
 <gazebo reference="left_wheel">
     <material>Gazebo/Purple</material>
@@ -224,6 +200,3 @@
     <material>Gazebo/Blue</material>
 </gazebo>
-<gazebo reference="camera_link_optical">
-    <material>Gazebo/Yellow</material>
-</gazebo>
 </robot>
